File: BendeRadio/BendeRadio.kicad_pcb (KiCad board)
At the start: 2 copper layers, 81.3 x 76.2 mm, 34 parts, among them J1 5V, J2 Conn_01x02, J3 Conn_01x02, J4 DISPLAY, J5 Encoder, J6 JTAG, U1 ESP32-WROOM-32, U2 Level shifter, U3 PAM8403 Amplifier, U4 PCM5102

Commit message: Revision 1.0.0
Parts:
- moved C10 1.27 mm to (97.8, 116.8), turned to -90 degrees
- moved J6 1.27 mm to (133.3, 104.1)
- moved C8 1.04 mm to (118.1, 57.4)
Routing:
- net /TCK: track 46.9 -> 51.9 mm
- net Net-(C1-Pad1): track 32.5 -> 35.1 mm
- net Net-(F1-OUT): track 22.7 -> 24.4 mm
- net /TMS: track 37.7 -> 36.4 mm
- net VCC: track 97.1 -> 98.1 mm
- net Net-(U1-G27): track 24.7 -> 25.5 mm
- net /TDI: track 39.0 -> 38.5 mm
- net /TDO: track 9.42 -> 9.94 mm
- net +3.3V: track 104.8 -> 105.3 mm
- net GND: track 27.8 -> 27.9 mm, vias 2 -> 3

Commit message: BendeRadio 1.1.0
Parts:
- moved C6 10.6 mm to (89.4, 109.7), turned to 90 degrees
- moved C10 8.07 mm to (105.7, 118.6), turned to 180 degrees
- moved U4 5.50 mm to (81.0, 116.8)
- moved F2 3.84 mm to (94.0, 101.1)
- moved C5 3.81 mm to (76.2, 101.6)
- moved REF** 1.80 mm to (114.0, 89.7)
- moved REF** 1.78 mm to (114.3, 82.0)
- moved C4 1.11 mm to (86.1, 94.2), turned to 180 degrees
- moved C13 0.51 mm to (63.0, 69.8)
Routing:
- net Net-(U3-in_left): track 54.2 -> 59.4 mm
- net +3.3V: track 105.3 -> 101.0 mm
- net Net-(J2-Pin_2): track 20.6 -> 23.9 mm
- net Net-(F2-OUT): track 28.0 -> 24.8 mm
- net Net-(U1-G25): track 31.0 -> 28.6 mm
- net Net-(U1-G27): track 25.5 -> 23.6 mm
- net /TMS: track 36.4 -> 37.9 mm
- net Net-(U1-G26): track 23.3 -> 21.9 mm
- net VCC: track 98.1 -> 99.5 mm
- net Net-(J3-Pin_2): track 18.6 -> 19.5 mm
- net Net-(F3-OUT): track 41.2 -> 42.0 mm
- net Net-(U3-in_right): track 26.3 -> 27.0 mm
- net Net-(U3-in_GND): track 26.3 -> 27.0 mm
- net GND: track 27.9 -> 28.6 mm, vias 3 -> 4
- net /TCK: track 51.9 -> 51.4 mm
